File: KiCad/i386sx-socket.kicad_pcb (KiCad board)
At the start: 2 copper layers, 38.1 x 38.1 mm, 14 parts, among them J1 CPU 1-25, J2 CPU 26-50, J3 CPU 51-75, J4 CPU 76-100, U1 80386SX/TI486SXLC/Cx486SLC, U2 NCP1117-3.3

Commit message: Make PCB slightly larger so that zones connect on the outside edge
Routing:
- net VCC: track 137.8 -> 283.8 mm
- net GND: track 256.9 -> 282.8 mm
Other:
- board size 38.1 x 38.1 mm -> 38.7 x 38.7 mm
- board text added: "V1.0"
